File: kicad/harite.kicad_sch (KiCad schematic)
At the start: 76 parts, among them J1 Cirque Connector, J2 Cirque Connector, U1 RP2040_Zero, U2 RP2040_Zero

Commit message: v2
Parts:
- removed D25, D26, D31, D32, D33, D34, D35, D36, D37, D38, D39, D40, D41, D42, D43, D44, D45, D46, D47, D48, D49, D50: D, ScottoKeebs_Components:Diode_SOD-123, symbol Device:D
- removed H10, H6, H7, H8, H9: Mounting_Hole, MountingHole:MountingHole_2.2mm_M2_Pad_Via, symbol ScottoKeebs:Placeholder_Mounting_Hole
- removed J1, J2: Cirque Connector, footprints:Cirque-connector, symbol Connector_Generic:Conn_01x06
- removed S10, S7, S8, S9: SKRHADE010, footprints:SKRHADE, symbol SKRHADE010:SKRHADE010
- removed U2: RP2040_Zero, ScottoKeebs_MCU:RP2040_Zero, symbol ScottoKeebs:MCU_RP2040_Zero
- removed USB2: HRO-TYPE-C-31-M-12, footprints:HRO-TYPE-C-31-M-12, symbol USBType-C:HRO-TYPE-C-31-M-12
- added D19, D20: D, ScottoKeebs_Components:Diode_SOD-123, symbol Device:D
- added J1: 59453-121110ECHLF, AMPHENOL_59453-121110ECHLF, symbol 59453-121110ECHLF:59453-121110ECHLF
- added J2, J3: 59453-051110ECHLF, AMPHENOL_59453-051110ECHLF, symbol 59453-051110ECHLF:59453-051110ECHLF
- added J4, J5: 59453-081110EDHLF, AMPHENOL_59453-081110EDHLF, symbol 59453-081110EDHLF:59453-081110EDHLF
- S1, S2, S3, S4, S5, S6: footprint footprints:SKRHADE -> SKRHADE010
- renumbered D19 to D25, D20 to D26
Connections:
- net RRow 4 is gone; now on net ERow 4: D29.1 (K)
- net RRow 5 is gone; now on net ERow 5: D30.1 (K)
- net 3V3: now also J1.1, J2.1
- net Col 1: now also U1.12 (11); no longer U1.10 (9)
- net Col 2: now also U1.13 (12); no longer U1.11 (10)
- net Col 3: now also U1.14 (13); no longer U1.12 (11)
- net Col 4: now also U1.15 (14); no longer U1.13 (12)
- net Col 5: now also U1.16 (15), J5.7; no longer S5.5 (COMMON), U1.14 (13)
- net GND: now also J1.2, J2.4
- net Row 1: now also U1.7 (6), J5.5; no longer D21.1 (K), U1.15 (14)
- net Row 2: now also U1.8 (7), J5.4; no longer D22.1 (K), U1.16 (15)
- net Row 3: now also U1.9 (8), J5.3; no longer D23.1 (K), U1.17 (26)
- net Row 4: now also U1.10 (9), J5.6; no longer D24.1 (K), U1.18 (27)
- net Row 5: now also U1.11 (10), J5.8; no longer U1.19 (28)
- net SCK: now also J1.12
- net SS: now also J1.10
- net at D23.2 (A): now also S6.2 (CENTER); no longer S5.3 (C)
- net at S5.2 (CENTER): now also D20.2 (A); no longer D22.2 (A)
- net at D21.2 (A): now also S5.3 (C); no longer S5.1 (A)
- net at D27.2 (A): now also S5.4 (B); no longer S6.2 (CENTER)
- net at D24.2 (A): now also S6.3 (C); no longer S5.4 (B)
- net at S5.6 (D): now also D28.2 (A)
- net JC: now reaches U1.20 (29)
- net JC: now also J2.3
- net at S6.1 (A): now also D22.2 (A)
- net RCol 1 renamed ECol 6
- net ECol 6: now also J4.7
- net RRow 2 renamed ERow 4
- net ERow 4: now also J4.3
- net RRow 3 renamed ERow 5
- net ERow 5: now also J4.1
- net SI renamed MOSI
- net MOSI: now also J1.8
- net SO renamed MISO
- net MISO: now also J1.11
- new net: D19.2 (A), S5.1 (A)
- new net Col 6: J5.2, U1.17 (26)
- new net E3V3: J3.5
- new net ECol 5: J4.2, S5.5 (COMMON)
- new net EGND: J3.2
- new net EJC: J3.3
- new net EJX: J3.1
- new net EJY: J3.4
- new net ERow 1: D19.1 (K), D22.1 (K), J4.4
- new net ERow 2: D20.1 (K), D23.1 (K), J4.5
- new net ERow 3: D21.1 (K), D24.1 (K), J4.6
- new net JX: J2.5, U1.18 (27)
- new net JY: J2.2, U1.19 (28)
