File: kicad/left/left.kicad_pcb (KiCad board)
At the start: 2 copper layers, 126 x 46.9 mm, 33 parts, among them J1 59453-121110ECHLF, J2 59453-051110ECHLF, J5 59453-081110EDHLF, U1 RP2040_Zero

Commit message: wiring
Parts:
- moved G*** 70.2 mm to (46.5, 90.5)
Connections:
- J2 pad 3: JC -> JX
- J2 pad 4: GND -> JC
- J2 pad 5: JX -> GND
Routing:
- net JX: track 22.2 -> 26.4 mm, vias 1 -> 2
- net JC: track 31.4 -> 29.0 mm
- net GP0: track 46.4 -> 44.1 mm
- net GND: track 9.94 -> 7.98 mm
- net Row 1: track 142.5 -> 144.2 mm
- net Row 5: track 140.3 -> 139.6 mm
Other:
- board size 126 x 46.9 mm -> 126 x 47.8 mm
