File: kicad/left/left.kicad_pcb (KiCad board)
At the start: 2 copper layers, 126 x 47.8 mm, 36 parts, among them J1 59453-121110ECHLF, J2 59453-051110ECHLF, J3 Conn_01x06_Pin, J4 Conn_01x05_Pin, J5 59453-081110EDHLF, U1 RP2040_Zero

Commit message: Add gerbers
Routing:
- net Row 4: track 137.5 -> 135.9 mm
- net Row 2: track 170.7 -> 169.2 mm
- net Row 1: track 144.9 -> 145.9 mm
- net GND: track 17.7 -> 18.5 mm
- net Row 5: track 138.6 -> 137.9 mm
- net Col 2: track 90.4 -> 90.1 mm, vias 5 -> 4
