File: kicad/thumb-cluster/thumb-cluster.kicad_pcb (KiCad board)
At the start: 2 copper layers, 21 x 45 mm, 15 parts, among them J4 59453-081110EDHLF

Commit message: wiring
Routing:
- net ERow 3: track 36.4 -> 34.6 mm, vias 2 -> 0
- net ERow 5: track 53.2 -> 51.6 mm
- net ECol 6: track 56.3 -> 54.9 mm
- net ERow 1: track 33.7 -> 32.5 mm
- net ECol 5: track 30.7 -> 31.3 mm
Other:
- outline, holes or cut-outs redrawn
