File: kicad/right/right.kicad_pcb (KiCad board)
At the start: 2 copper layers, 126 x 47.8 mm, 36 parts, among them J1 59453-121110ECHLF, J2 59453-051110ECHLF, J3 Conn_01x06_Pin, J4 Conn_01x05_Pin, J5 59453-081110EDHLF, U1 RP2040_Zero

Commit message: place right components
Parts:
- removed the G*** at (46.5, 90.5)
- added G***: LOGO, footprints:logo-right, F.Cu at (250.5, 90.5)
- moved H1 249.7 mm to (273.4, 103.2)
- moved H4 249.7 mm to (273.4, 84.7)
- moved D3 236.3 mm to (260.7, 103.3), turned to 45 degrees
- moved D5 236.2 mm to (272.1, 91.8), turned to -135 degrees
- moved S1 233.5 mm to (265.2, 96.1), turned to 45 degrees
- moved D4 231.8 mm to (269.7, 89.5), turned to -135 degrees
- moved D2 231.7 mm to (258.1, 101.8), turned to 45 degrees
- moved D1 227.7 mm to (256.1, 100.1), turned to 45 degrees
- moved D8 187.3 mm to (236.1, 90.4), turned to 45 degrees
- moved D10 186.1 mm to (246.9, 77.2), turned to -135 degrees
- moved D7 183.6 mm to (234.3, 88.6), turned to 45 degrees
- moved S2 183.5 mm to (240.2, 82.1), turned to 45 degrees
- moved D9 181.9 mm to (244.7, 75.3), turned to -135 degrees
- moved D6 179.7 mm to (232.5, 86.7), turned to 45 degrees
- moved J3 156.0 mm to (227.5, 82.8)
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Routing:
- net Row 3: track 182.6 -> 0.00 mm, vias 8 -> 0
- net Row 2: track 170.7 -> 0.00 mm, vias 10 -> 0
- net Row 1: track 144.9 -> 0.00 mm, vias 2 -> 0
- net Row 5: track 138.6 -> 0.00 mm, vias 8 -> 0
- net Row 4: track 137.5 -> 0.00 mm, vias 4 -> 0
- net Col 1: track 124.1 -> 0.00 mm, vias 2 -> 0
- net 3V3: track 106.8 -> 0.00 mm, vias 2 -> 0
- net Col 2: track 90.4 -> 0.00 mm, vias 5 -> 0
- net MOSI: track 85.4 -> 0.00 mm, vias 1 -> 0
- net SS: track 80.8 -> 0.00 mm, vias 1 -> 0
- net MISO: track 78.6 -> 0.00 mm, vias 3 -> 0
- net SCK: track 78.2 -> 0.00 mm, vias 1 -> 0
- net Col 3: track 64.6 -> 0.00 mm, vias 3 -> 0
- net 5V: track 64.1 -> 0.00 mm
- net GP0: track 44.1 -> 0.00 mm, vias 1 -> 0
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Other:
- board size 126 x 47.8 mm -> 258 x 47.9 mm

Commit message: wire right
Parts:
- moved D1 1.69 mm to (257.7, 99.7)
- moved D2 1.50 mm to (259.5, 101.4)
- moved D11 1.31 mm to (207.7, 82.8)
- moved D6 1.03 mm to (233.5, 86.7)
- moved D15 1.02 mm to (221.9, 74.5)
- moved D7 1.02 mm to (235.3, 88.4)
- moved D8 1.02 mm to (237.1, 90.2)
- moved D12 1.01 mm to (209.7, 84.7)
- moved D13 0.85 mm to (211.7, 86.7)
- moved D16 0.73 mm to (182.5, 91.6)
- moved D3 0.67 mm to (261.3, 103.2)
- moved D17 0.63 mm to (184.5, 93.6)
- moved D14 0.63 mm to (219.7, 72.2)
- moved D18 0.49 mm to (186.5, 95.6)
- moved D10 0.40 mm to (246.9, 77.7)
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- renumbered G*** to ?
Routing:
- net Row 5: track 0.00 -> 157.0 mm, vias 0 -> 7
- net 3V3: track 0.00 -> 151.8 mm, vias 0 -> 1
- net Row 4: track 0.00 -> 144.9 mm, vias 0 -> 9
- net Row 1: track 0.00 -> 141.6 mm, vias 0 -> 7
- net Row 2: track 0.00 -> 139.4 mm, vias 0 -> 6
- net Row 3: track 0.00 -> 136.8 mm, vias 0 -> 4
- net Col 1: track 0.00 -> 131.3 mm, vias 0 -> 2
- net Col 2: track 0.00 -> 103.6 mm
- net SCK: track 0.00 -> 86.9 mm, vias 0 -> 1
- net MISO: track 0.00 -> 85.1 mm, vias 0 -> 1
- net Col 3: track 0.00 -> 82.1 mm
- net SS: track 0.00 -> 81.8 mm, vias 0 -> 1
- net MOSI: track 0.00 -> 81.6 mm, vias 0 -> 1
- net Col 4: track 0.00 -> 61.3 mm
- net 5V: track 0.00 -> 46.7 mm
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Other:
- board size 258 x 47.9 mm -> 126 x 47.9 mm

Commit message: Add gerbers
Routing:
- net Row 1: track 141.6 -> 139.3 mm
- net Row 5: track 157.0 -> 155.7 mm
- net GND: track 18.1 -> 17.4 mm
- net Net-(D8-A): track 4.05 -> 4.58 mm
